File: espflie-cam-deck.sch (KiCad schematic (older format))
At the start: 83 parts, among them J1 Conn_01x02, J10 Conn_01x02, J11 Conn_01x02, J12 Conn_01x26, J4 Conn_01x08, J5 Conn_01x08, J6 Conn_01x02, J7 Conn_01x02, Q1 AO3401A, Q2 AO3400A, Q3 AO3400A, Q4 AO3400A, Q5 AO3400A, SW1 SW_MEC_5E, SW2 SW_MEC_5E, U1 BC847BDW1T1G, U2 USB_C_16_PIN, U3 MPU-6050, U4 ME6211C33M5G-N, U5 CP2102N-A01-GQFN28, U6 ESP-PSRAM32, U7 ME6211C28M5G-N, U8 ME6211C15M5G-N

Commit message: .
Parts:
- removed C1: 10nF, Capacitor_SMD:C_0402_1005Metric, symbol Device:C
- removed C2, C4: 0.1uF, Capacitor_SMD:C_0402_1005Metric, symbol Device:C
- removed C5: 2.2nF, Capacitor_SMD:C_0402_1005Metric, symbol Device:C
- removed D1: LED-WHT, LED_SMD:LED_0402_1005Metric, symbol Device:LED
- removed D2: LED-BLE, LED_SMD:LED_0402_1005Metric, symbol Device:LED
- removed D3: LED-RED, LED_SMD:LED_0402_1005Metric, symbol Device:LED
- removed D4: LED-GRN, LED_SMD:LED_0402_1005Metric, symbol Device:LED
- removed D6, D7, D8, D9: 1N4148WT, Diode_SMD:D_SOD-523, symbol Diode:1N4148WT
- removed J10, J11, J6, J7: Conn_01x02, Connector_JST:JST_PH_S2B-PH-K_1x02_P2.00mm_Horizontal, symbol Connector_Generic:Conn_01x02
- removed J4, J5: Conn_01x08, Connector_PinHeader_2.54mm:PinHeader_1x08_P2.54mm_Vertical_SMD_Pin1Right, symbol Connector_Generic:Conn_01x08
- removed Q2, Q3, Q4, Q5: AO3400A, Package_TO_SOT_SMD:SOT-23, symbol Transistor_FET:AO3400A
- removed R10, R14, R15, R16, R18, R19, R21, R22, R7: 10K, Resistor_SMD:R_0402_1005Metric, symbol Device:R
- removed R20: 0R, Resistor_SMD:R_0402_1005Metric, symbol Device:R
- removed R4, R5: 82K, Resistor_SMD:R_0402_1005Metric, symbol Device:R
- removed R8: 2K, Resistor_SMD:R_0402_1005Metric, symbol Device:R
- removed R9: 3K, Resistor_SMD:R_0402_1005Metric, symbol Device:R
- removed U3: MPU-6050, Sensor_Motion:InvenSense_QFN-24_4x4mm_P0.5mm, symbol Sensor_Motion:MPU-6050
- C1: renamed from R3; symbol Device:R -> Device:C
- U1: renamed from U4; value ME6211C33M5G-N -> ME6217C33M5G; symbol LDO:ME6211C33M5G-N -> LDO:ME6217C33M5G
- renumbered C12 to C10, C13 to C11, C15 to C12, C14 to C13, C17 to C14, C18 to C15, C19 to C16, C20 to C17, C3 to C2, C7 to C3, C8 to C4, C6 to C5, C9 to C6, C16 to C7, C10 to C8, C11 to C9, D5 to D1, J12 to J2, R25 to R10, R26 to R11, R27 to R12, R28 to R13, R6 to R3, R13 to R4, R11 to R5, R12 to R6, R17 to R7, R23 to R8, R24 to R9, U1 to U3, U6 to U4, U7 to U6, U8 to U7
Connections:
- net GNDA is gone; now on net GND: C8.2, J2.2 (Pin_2)
- net +3V3: now also C5.2, C6.2; no longer C5.1, C6.1
- net GND: now also C5.1, C6.1; no longer C5.2, C6.2
- net VCC: now reaches U1.4 (VIN)
- net VCC: now also C14.1, C15.1, C2.1, D1.1 (K), Q1.2 (S), U1.1 (CE), U6.1 (VIN), U6.3 (EN), U7.1 (VIN), U7.3 (EN)
- removed net VSS: C14.1, C15.1, C2.1, D1.1 (K), Q1.2 (S), U1.1 (VIN), U1.3 (EN), U6.1 (VIN), U6.3 (EN), U7.1 (VIN), U7.3 (EN)
- no-connect marks 30 -> 32
Other:
- moved on the sheet: AE1, C10, C11, C12, C13, C14, C15, C16, C17, C2, C3, C4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
